File: hardware/monosplit/pcb/awkb_monosplit.kicad_pcb (KiCad board)
At the start: 2 copper layers, 245.6 x 120.1 mm, 94 parts, among them J1 Conn_01x12_Socket, J2 Conn_01x06_Female, J3 OLED, J4 Conn_01x04_Socket, J5 Conn_01x04_Socket, SW1 SW1, SW10 SW10, SW11 SW11, SW12 SW12, SW13 SW13, SW14 SW14, SW15 SW15, SW16 SW16, SW17 SW17, SW18 SW18, SW19 SW19, SW2 SW2, SW20 SW20, SW21 SW21, SW22 SW22, SW23 SW23, SW24 SW24, SW25 SW25, SW26 SW26, SW27 SW27, SW28 SW28, SW29 SW29, SW3 SW3, SW30 SW30, SW31 SW31, SW32 SW32, SW33 SW33, SW34 SW34, SW4 SW4, SW5 SW5, SW6 SW6, SW7 SW7, SW8 SW8, SW9 SW9, U1 ProMicro

Commit message: Non-essential change in firmware; Modified monosplit hardward
Parts:
- removed G***: LOGO, jw_custom_image:squares_multi_1_9x9_13mm
- removed J2: Conn_01x06_Female, Connector_FFC-FPC:Hirose_FH12-6S-0.5SH_1x06-1MP_P0.50mm_Horizontal
- removed MH1, MH2: MCU, MountingHole:MountingHole_2.2mm_M2_ISO7380_Pad
- removed the TRH1 at (137.1, 74.0)
- removed the TRH2 at (162.9, 74.0)
- removed the TRH3 at (164.2, 130.4)
- removed the TRH4 at (135.8, 130.4)
- added J4: OLED, Connector_PinSocket_2.54mm:PinSocket_1x04_P2.54mm_Vertical, F.Cu at (167.4, 109.6)
- added OH3: OLED cover, MountingHole:MountingHole_2.2mm_M2_ISO7380_Pad, F.Cu at (171.4, 109.6)
- added OH4: OLED cover, MountingHole:MountingHole_2.2mm_M2_ISO7380_Pad, F.Cu at (128.4, 109.6)
- added R1: 4.7k, Resistor_SMD:R_1206_3216Metric_Pad1.30x1.75mm_HandSolder, F.Cu at (162.0, 80.2)
- added R2: 4.7k, Resistor_SMD:R_1206_3216Metric_Pad1.30x1.75mm_HandSolder, F.Cu at (162.0, 82.7)
- added TRH1: Trackpad, MountingHole:MountingHole_2.2mm_M2_ISO7380_Pad, F.Cu at (32.3, 124.1)
- added TRH1: Trackpad, MountingHole:MountingHole_2.2mm_M2_ISO7380_Pad, F.Cu at (137.1, 140.6)
- added TRH1: Trackpad, MountingHole:MountingHole_2.2mm_M2_ISO7380_Pad, F.Cu at (138.0, 64.2)
- added TRH2: Trackpad, MountingHole:MountingHole_2.2mm_M2_ISO7380_Pad, F.Cu at (161.1, 140.7)
- added TRH2: Trackpad, MountingHole:MountingHole_2.2mm_M2_ISO7380_Pad, F.Cu at (162.0, 64.2)
- added TRH2: Trackpad, MountingHole:MountingHole_2.2mm_M2_ISO7380_Pad, F.Cu at (56.3, 124.2)
- added TRH3: Trackpad, MountingHole:MountingHole_2.2mm_M2_ISO7380_Pad, F.Cu at (161.1, 182.2)
- added TRH3: Trackpad, MountingHole:MountingHole_2.2mm_M2_ISO7380_Pad, F.Cu at (162.0, 105.8)
- added TRH3: Trackpad, MountingHole:MountingHole_2.2mm_M2_ISO7380_Pad, F.Cu at (56.3, 165.7)
- added TRH4: Trackpad, MountingHole:MountingHole_2.2mm_M2_ISO7380_Pad, F.Cu at (137.1, 182.2)
- added TRH4: Trackpad, MountingHole:MountingHole_2.2mm_M2_ISO7380_Pad, F.Cu at (138.0, 105.8)
- added TRH4: Trackpad, MountingHole:MountingHole_2.2mm_M2_ISO7380_Pad, F.Cu at (32.3, 165.7)
- added TRH5: Trackpad, MountingHole:MountingHole_2.2mm_M2_ISO7380_Pad, F.Cu at (138.0, 90.2)
- added TRH5: Trackpad, MountingHole:MountingHole_2.2mm_M2_ISO7380_Pad, F.Cu at (77.3, 182.5)
- added TRH5: Trackpad, MountingHole:MountingHole_2.2mm_M2_ISO7380_Pad, F.Cu at (77.3, 156.5)
- added TRH6: Trackpad, MountingHole:MountingHole_2.2mm_M2_ISO7380_Pad, F.Cu at (162.0, 90.1)
- added TRH6: Trackpad, MountingHole:MountingHole_2.2mm_M2_ISO7380_Pad, F.Cu at (101.3, 182.4)
- added TRH6: Trackpad, MountingHole:MountingHole_2.2mm_M2_ISO7380_Pad, F.Cu at (101.3, 156.5)
- J6: renamed from J4; moved to B.Cu
- moved OH1 48.7 mm to (207.5, 23.6), turned to 105 degrees
- moved OH2 41.1 mm to (167.8, 41.5), turned to 105 degrees
- moved J3 37.4 mm to (205.5, 31.7), turned to -165 degrees
- moved D32 25.1 mm to (125.8, 116.9), turned to 90 degrees
- moved J1 23.4 mm to (133.7, 81.1)
- moved D33 22.7 mm to (175.3, 119.1), turned to -90 degrees
- moved D31 21.5 mm to (109.3, 110.5), turned to -90 degrees
- moved D34 20.4 mm to (190.8, 112.0), turned to 90 degrees
- moved D25 17.1 mm to (121.9, 97.5), turned to 90 degrees
- moved D15 16.8 mm to (126.3, 79.0), turned to 90 degrees
- moved D5 16.6 mm to (130.7, 60.6), turned to 90 degrees
- moved D24 16.3 mm to (104.3, 89.7), turned to -90 degrees
- moved D14 16.0 mm to (108.4, 71.2), turned to -90 degrees
- moved D23 15.9 mm to (86.5, 82.0), turned to 90 degrees
- moved D4 15.7 mm to (113.1, 52.7), turned to -90 degrees
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Connections:
- D10 pad 1: row0 -> Net-(D10-K)
- D10 pad 2: Net-(D10-A) -> row0
- D16 pad 1: row1 -> Net-(D16-K)
- D16 pad 2: Net-(D16-A) -> row1
- D17 pad 1: Net-(D17-K) -> row1
- D17 pad 2: row1 -> Net-(D17-A)
- D18 pad 1: row1 -> Net-(D18-K)
- D18 pad 2: Net-(D18-A) -> row1
- D19 pad 1: Net-(D19-K) -> row1
- D19 pad 2: row1 -> Net-(D19-A)
- D20 pad 1: row1 -> Net-(D20-K)
- D20 pad 2: Net-(D20-A) -> row1
- D26 pad 1: row2 -> Net-(D26-K)
- D26 pad 2: Net-(D26-A) -> row2
- D27 pad 1: Net-(D27-K) -> row2
- D27 pad 2: row2 -> Net-(D27-A)
- D28 pad 1: row2 -> Net-(D28-K)
- D28 pad 2: Net-(D28-A) -> row2
- D29 pad 1: Net-(D29-K) -> row2
- D29 pad 2: row2 -> Net-(D29-A)
- D30 pad 1: row2 -> Net-(D30-K)
- D30 pad 2: Net-(D30-A) -> row2
- D33 pad 1: Net-(D33-K) -> row3
- D33 pad 2: row3 -> Net-(D33-A)
- D34 pad 1: row3 -> Net-(D34-K)
- D34 pad 2: Net-(D34-A) -> row3
- D6 pad 1: row0 -> Net-(D6-K)
- D6 pad 2: Net-(D6-A) -> row0
- D7 pad 1: Net-(D7-K) -> row0
- D7 pad 2: row0 -> Net-(D7-A)
- D8 pad 1: row0 -> Net-(D8-K)
- D8 pad 2: Net-(D8-A) -> row0
- D9 pad 1: Net-(D9-K) -> row0
- D9 pad 2: row0 -> Net-(D9-A)
- J1 pad 3: unconnected-(J1-Pin_3-Pad3) -> SDA
- J1 pad 4: unconnected-(J1-Pin_4-Pad4) -> SCL
- J3 pad 1: SDA -> SDA_conn
- J3 pad 2: SCL -> SCL_conn
- J3 pad 3: VCC -> VCC_conn
- J3 pad 4: GND -> GND_conn
- J5 pad 1: GND -> SDA
- J5 pad 2: VCC -> SCL
- J5 pad 3: SCL -> VCC
- J5 pad 4: SDA -> GND
- J6 pad 1: SDA -> SDA_conn
- J6 pad 2: SCL -> SCL_conn
- J6 pad 3: VCC -> VCC_conn
- J6 pad 4: GND -> GND_conn
- SW10 pad 1: Net-(D10-A) -> col4
- SW10 pad 2: col4 -> Net-(D10-K)
- SW16 pad 1: Net-(D16-A) -> col2
- SW16 pad 2: col2 -> Net-(D16-K)
- SW17 pad 1: col3 -> Net-(D17-A)
- SW17 pad 2: Net-(D17-K) -> col3
- SW18 pad 1: Net-(D18-A) -> col3
- SW18 pad 2: col3 -> Net-(D18-K)
- SW19 pad 1: col4 -> Net-(D19-A)
- SW19 pad 2: Net-(D19-K) -> col4
- SW20 pad 1: Net-(D20-A) -> col4
- SW20 pad 2: col4 -> Net-(D20-K)
- SW26 pad 1: Net-(D26-A) -> col2
- SW26 pad 2: col2 -> Net-(D26-K)
- SW27 pad 1: col3 -> Net-(D27-A)
- SW27 pad 2: Net-(D27-K) -> col3
- SW28 pad 1: Net-(D28-A) -> col3
- SW28 pad 2: col3 -> Net-(D28-K)
- SW29 pad 1: col4 -> Net-(D29-A)
- SW29 pad 2: Net-(D29-K) -> col4
- SW30 pad 1: Net-(D30-A) -> col4
- SW30 pad 2: col4 -> Net-(D30-K)
- SW33 pad 1: col3 -> Net-(D33-A)
- SW33 pad 2: Net-(D33-K) -> col3
- SW34 pad 1: Net-(D34-A) -> col3
- SW34 pad 2: col3 -> Net-(D34-K)
- SW6 pad 1: Net-(D6-A) -> col2
- SW6 pad 2: col2 -> Net-(D6-K)
- SW7 pad 1: col3 -> Net-(D7-A)
- SW7 pad 2: Net-(D7-K) -> col3
- SW8 pad 1: Net-(D8-A) -> col3
- SW8 pad 2: col3 -> Net-(D8-K)
- SW9 pad 1: col4 -> Net-(D9-A)
- SW9 pad 2: Net-(D9-K) -> col4
- U1 pad 10: row1 -> col4
- U1 pad 11: row2 -> col3
- U1 pad 13: col0 -> col2
- U1 pad 17: col1 -> unconnected-(U1-A0(PF7)-Pad17)
- U1 pad 18: col2 -> unconnected-(U1-A1(PF6)-Pad18)
- U1 pad 19: col3 -> col1
- U1 pad 20: col4 -> col0
- U1 pad 7: unconnected-(U1-D4(PD4)-Pad7) -> row0
- U1 pad 8: unconnected-(U1-D5(PC6)-Pad8) -> row1
- U1 pad 9: row0 -> row2
Routing:
- net row2: track 0.00 -> 236.5 mm, vias 0 -> 3
- net row0: track 0.00 -> 233.5 mm, vias 0 -> 3
- net row1: track 0.00 -> 216.9 mm, vias 0 -> 1
- net col1: track 0.00 -> 186.3 mm, vias 0 -> 6
- net col3: track 0.00 -> 164.2 mm, vias 0 -> 5
- net col0: track 0.00 -> 161.7 mm, vias 0 -> 5
- net col4: track 0.00 -> 154.3 mm, vias 0 -> 4
- net col2: track 0.00 -> 141.6 mm, vias 0 -> 6
- net row3: track 0.00 -> 123.5 mm, vias 0 -> 4
- net SDA: track 28.8 -> 108.4 mm, vias 0 -> 3
- net SCL: track 28.2 -> 106.9 mm, vias 0 -> 3
- net VCC: track 75.1 -> 115.7 mm, vias 3 -> 5
- net GND: track 32.7 -> 3.47 mm
- net NCS: track 0.00 -> 28.8 mm, vias 0 -> 1
- net MOSI: track 0.00 -> 22.8 mm
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Other:
- board size 245.6 x 120.1 mm -> 249.5 x 166.6 mm
- board text added: "Cirque Trackpad TM023023"
