File: hardware/monosplit/pcb/awkb_monosplit.kicad_sch (KiCad schematic)
At the start: 93 parts, among them J1 Conn_01x12_Socket, J2 Conn_01x06_Female, J3 OLED, J4 Conn_01x04_Socket, J5 Conn_01x04_Socket, SW1 ${REFERENCE}, SW10 ${REFERENCE}, SW11 ${REFERENCE}, SW12 ${REFERENCE}, SW13 ${REFERENCE}, SW14 ${REFERENCE}, SW15 ${REFERENCE}, SW16 ${REFERENCE}, SW17 ${REFERENCE}, SW18 ${REFERENCE}, SW19 ${REFERENCE}, SW2 ${REFERENCE}, SW20 ${REFERENCE}, SW21 ${REFERENCE}, SW22 ${REFERENCE}, SW23 ${REFERENCE}, SW24 ${REFERENCE}, SW25 ${REFERENCE}, SW26 ${REFERENCE}, SW27 ${REFERENCE}, SW28 ${REFERENCE}, SW29 ${REFERENCE}, SW3 ${REFERENCE}, SW30 ${REFERENCE}, SW31 ${REFERENCE}, SW32 ${REFERENCE}, SW33 ${REFERENCE}, SW34 ${REFERENCE}, SW4 ${REFERENCE}, SW5 ${REFERENCE}, SW6 ${REFERENCE}, SW7 ${REFERENCE}, SW8 ${REFERENCE}, SW9 ${REFERENCE}, U1 ProMicro

Commit message: Non-essential change in firmware; Modified monosplit hardward
Parts:
- removed J2: Conn_01x06_Female, Connector_FFC-FPC:Hirose_FH12-6S-0.5SH_1x06-1MP_P0.50mm_Horizontal, symbol Connector:Conn_01x06_Female
- removed J4: Conn_01x04_Socket, Connector_FFC-FPC:Molex_200528-0040_1x04-1MP_P1.00mm_Horizontal, symbol Connector:Conn_01x04_Socket
- removed MH1, MH2: MCU, MountingHole:MountingHole_2.2mm_M2_ISO7380_Pad, symbol SofleKeyboard-rescue:HOLE-Lily58-cache-Lily58_Pro-rescue
- added J4: OLED, Connector_PinSocket_2.54mm:PinSocket_1x04_P2.54mm_Vertical, symbol SofleKeyboard-rescue:OLED-Lily58-cache-Lily58_Pro-rescue
- added J6: Conn_01x04_Socket, Connector_FFC-FPC:Molex_200528-0040_1x04-1MP_P1.00mm_Horizontal, symbol Connector:Conn_01x04_Socket
- added OH3, OH4: OLED cover, MountingHole:MountingHole_2.2mm_M2_ISO7380_Pad, symbol SofleKeyboard-rescue:HOLE-Lily58-cache-Lily58_Pro-rescue
- added R1, R2: 4.7k, Resistor_SMD:R_1206_3216Metric_Pad1.30x1.75mm_HandSolder, symbol Device:R
- added TRH5, TRH6: Trackpad, MountingHole:MountingHole_2.2mm_M2_ISO7380_Pad, symbol SofleKeyboard-rescue:HOLE-Lily58-cache-Lily58_Pro-rescue
Connections:
- net GND: now also J5.4 (Pin_4), J4.4 (P4); no longer J3.4 (P4), J5.1 (Pin_1)
- net SCL: now also J1.4 (Pin_4), J5.2 (Pin_2), J4.2 (P2), R2.1; no longer J3.2 (P2), J5.3 (Pin_3)
- net SDA: now also J1.3 (Pin_3), J5.1 (Pin_1), J4.1 (P1), R1.1; no longer J3.1 (P1), J5.4 (Pin_4)
- net VCC: now also J5.3 (Pin_3), J4.3 (P3), R1.2, R2.2; no longer J3.3 (P3), J5.2 (Pin_2)
- net col0: now also U1.20 (A3(PF4)); no longer U1.13 (D10(PB6))
- net col1: now also U1.19 (A2(PF5)); no longer U1.17 (A0(PF7))
- net col2: now also SW16.1, SW26.1, SW6.1, U1.13 (D10(PB6)); no longer SW16.2, SW26.2, SW6.2, U1.18 (A1(PF6))
- net col3: now also SW17.2, SW18.1, SW27.2, SW28.1, SW33.2, SW34.1, SW7.2, SW8.1, U1.11 (D8(PB4)); no longer SW17.1, SW18.2, SW27.1, SW28.2, SW33.1, SW34.2, SW7.1, SW8.2, U1.19 (A2(PF5))
- net col4: now also SW10.1, SW19.2, SW20.1, SW29.2, SW30.1, SW9.2, U1.10 (D7(PE6)); no longer SW10.2, SW19.1, SW20.2, SW29.1, SW30.2, SW9.1, U1.20 (A3(PF4))
- net row0: now also D10.2 (A), D6.2 (A), D7.1 (K), D8.2 (A), D9.1 (K), U1.7 (D4(PD4)); no longer D10.1 (K), D6.1 (K), D7.2 (A), D8.1 (K), D9.2 (A), U1.9 (D6(PD7))
- net row1: now also D16.2 (A), D17.1 (K), D18.2 (A), D19.1 (K), D20.2 (A), U1.8 (D5(PC6)); no longer D16.1 (K), D17.2 (A), D18.1 (K), D19.2 (A), D20.1 (K), U1.10 (D7(PE6))
- net row2: now also D26.2 (A), D27.1 (K), D28.2 (A), D29.1 (K), D30.2 (A), U1.9 (D6(PD7)); no longer D26.1 (K), D27.2 (A), D28.1 (K), D29.2 (A), D30.1 (K), U1.11 (D8(PB4))
- net row3: now also D33.1 (K), D34.2 (A); no longer D33.2 (A), D34.1 (K)
- new net: D7.2 (A), SW7.1
- new net: D30.1 (K), SW30.2
- new net: D17.2 (A), SW17.1
- new net: D29.2 (A), SW29.1
- new net: D34.1 (K), SW34.2
- new net: D8.1 (K), SW8.2
- new net: D16.1 (K), SW16.2
- new net: D20.1 (K), SW20.2
- new net: D18.1 (K), SW18.2
- new net: D33.2 (A), SW33.1
- new net: D9.2 (A), SW9.1
- new net: D6.1 (K), SW6.2
- new net: D19.2 (A), SW19.1
- new net: D28.1 (K), SW28.2
- new net: D27.2 (A), SW27.1
- new net: D10.1 (K), SW10.2
- new net: D26.1 (K), SW26.2
- new net GND_conn: J3.4 (P4), J6.4 (Pin_4)
- new net SCL_conn: J3.2 (P2), J6.2 (Pin_2)
- new net SDA_conn: J3.1 (P1), J6.1 (Pin_1)
- new net VCC_conn: J3.3 (P3), J6.3 (Pin_3)
- no-connect marks 4 -> 1
Other:
- moved on the sheet: D1, D10, D11, D12, D13, D14, D15, D16, D17, D18, D19, D2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
