File: hardware/34 monosplit/pcb/awkb_monosplit.kicad_pcb (KiCad board)
At the start: 2 copper layers, 249.5 x 166.6 mm, 109 parts, among them J1 Conn_01x12_Socket, J3 OLED, J4 OLED, J5 Conn_01x04_Socket, J6 Conn_01x04_Socket, SW1 SW1, SW10 SW10, SW11 SW11, SW12 SW12, SW13 SW13, SW14 SW14, SW15 SW15, SW16 SW16, SW17 SW17, SW18 SW18, SW19 SW19, SW2 SW2, SW20 SW20, SW21 SW21, SW22 SW22, SW23 SW23, SW24 SW24, SW25 SW25, SW26 SW26, SW27 SW27, SW28 SW28, SW29 SW29, SW3 SW3, SW30 SW30, SW31 SW31, SW32 SW32, SW33 SW33, SW34 SW34, SW4 SW4, SW5 SW5, SW6 SW6, SW7 SW7, SW8 SW8, SW9 SW9, U1 ProMicro

Commit message: Re-organized hardware directory.. again
Parts:
- removed the TRH1 at (32.3, 124.1)
- removed the TRH1 at (137.1, 140.6)
- removed the TRH2 at (161.1, 140.7)
- removed the TRH2 at (56.3, 124.2)
- removed the TRH3 at (161.1, 182.2)
- removed the TRH3 at (56.3, 165.7)
- removed the TRH4 at (137.1, 182.2)
- removed the TRH4 at (32.3, 165.7)
- TRH1, TRH2, TRH3, TRH4, TRH5 (x3), TRH6 (x3): footprint MountingHole:MountingHole_2.2mm_M2_ISO7380_Pad -> MountingHole:MountingHole_3.2mm_M3
- moved TRH5 173.1 mm to (245.8, 143.2)
- moved TRH5 173.1 mm to (245.8, 117.2)
- moved TRH6 173.1 mm to (269.8, 143.1)
- moved TRH6 173.1 mm to (269.8, 117.2)
- moved OH4 9.50 mm to (128.4, 100.1)
- moved OH3 9.50 mm to (171.4, 100.1)
- moved H1 0.21 mm to (82.3, 111.7)
Routing:
- net row2: track 236.5 -> 239.6 mm
- net row3: track 123.5 -> 126.3 mm
- net GND: track 3.47 -> 1.54 mm, vias 2 -> 1
Other:
- board size 249.5 x 166.6 mm -> 248.3 x 126.5 mm
